Commit message: removing some refs to swarmfarm

File: urdf/swarm_farm.urdf (robot description, URDF)
Before this commit: robot swarm_farm, 6 links, 5 joints
Links:
- link back_chassis_link: geometry collision mesh filename=package://sprayerbot/meshes/swarmfarmv2_Body.dae; collision mesh filename=package://sprayerbot/meshes/swarmfarmv2_back_chassis_body.d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
- link back_left_wheel_link: geometry collision mesh filename=package://sprayerbot/meshes/swarmfarmv2_wheel_body.dae; visual mesh filename=package://sprayerbot/meshes/swarmfarmv2_wheel_body.dae
- link back_right_wheel_link: geometry collision mesh filename=package://sprayerbot/meshes/swarmfarmv2_wheel_body.dae; visual mesh filename=package://sprayerbot/meshes/swarmfarmv2_wheel_body.dae
- link front_chassis_link: geometry collision mesh filename=package://sprayerbot/meshes/swarmfarmv2_front_chassis_body.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; visual mesh filename=package://sprayerbot/meshes/swarmfarmv2_front_chassis_body.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
- link front_left_wheel_link: geometry collision mesh filename=package://sprayerbot/meshes/swarmfarmv2_wheel_body.dae; visual mesh filename=package://sprayerbot/meshes/swarmfarmv2_wheel_body.dae
- link front_right_wheel_link: geometry collision mesh filename=package://sprayerbot/meshes/swarmfarmv2_wheel_body.dae; visual mesh filename=package://sprayerbot/meshes/swarmfarmv2_wheel_body.dae
