Commit message: Adjusting for runinng in ros rolling and gz harmonic

File: robot_description/sprayer.urdf.xacro (robot description, xacro)
@@ -41,11 +41,4 @@
       <geometry>
         <mesh filename="file://$(find sprayerbot)/robot_description/meshes/swarmfarmv2_spray_boom.dae"/>
-      </geometry>
-    </visual>
-    <visual>
-      <!--back_chassis_part/Body005.-->
-      <origin rpy="0.0 -0.0 0.0" xyz="0.0 0.0 0.0"/>
-      <geometry>
-        <mesh filename="file://$(find sprayerbot)/robot_description/meshes/swarmfarmv2_Body.dae"/>
       </geometry>
     </visual>
@@ -126,17 +119,13 @@
   </ros2_control>
   <gazebo>
-    <plugin filename="ign_ros2_control-system" name="ign_ros2_control::IgnitionROS2ControlPlugin">
+    <plugin filename="gz_ros2_control-system" name="gz_ros2_control::GazeboSimROS2ControlPlugin">
       <ros>
         <remapping>diff_drive_base_controller/odometry:=odom</remapping>
         <remapping>diff_drive_base_controller/tf_odometry:=tf</remapping>
         <remapping>diff_drive_base_controller/cmd_vel_unstamped:=cmd_vel</remapping>
+        <remapping>/controller_manager/robot_description:=/robot_description</remapping>
       </ros>
       <parameters>$(find sprayerbot)/config/diffdrive_control.yaml</parameters>
     </plugin>
-    <plugin filename="ignition-gazebo-imu-system" name="gz::sim::systems::Imu">
-    </plugin>
-    <plugin filename="ignition-gazebo-sensors-system" name="ignition::gazebo::systems::Sensors">
-      <render_engine>ogre2</render_engine>
-    </plugin>
   </gazebo>
 </robot>

Commit message: Adding robot localization system

File: robot_description/sprayer.urdf.xacro (robot description, xacro)
@@ -2,4 +2,10 @@
 <robot xmlns:xacro="http://www.ros.org/wiki/xacro" name="swarm_farm">
   <xacro:include filename="$(find krytn)/robot_description/magni/inertial.xacro" />
+  <link name="base_link" />
+  <joint name="chassis_joint" type="fixed">
+    <child link="front_chassis_link"/>
+    <parent link="base_link"/>
+    <origin rpy="0.0 -0.0 0.0" xyz="0.0 0.0 0.0"/>
+  </joint>
   <!--Generated by CROSS, a ROS Workbench for FreeCAD (https://github.com/galou/freecad.cross)-->
   <link name="front_chassis_link">
@@ -121,6 +127,6 @@
     <plugin filename="gz_ros2_control-system" name="gz_ros2_control::GazeboSimROS2ControlPlugin">
       <ros>
-        <remapping>/diff_drive_base_controller/odometry:=odom</remapping>
-        <remapping>/diff_drive_base_controller/tf_odometry:=tf</remapping>
+        <!--  <remapping>/diff_drive_base_controller/odometry:=odom</remapping>
+        <remapping>/diff_drive_base_controller/tf_odometry:=tf</remapping> -->
         <remapping>/diff_drive_base_controller/cmd_vel_unstamped:=cmd_vel</remapping>
         <remapping>/controller_manager/robot_description:=/robot_description</remapping>

Commit message: setting up filters for gps based localization fusion with onboard odometry

File: robot_description/sprayer.urdf.xacro (robot description, xacro)
@@ -3,5 +3,5 @@
   <xacro:include filename="$(find krytn)/robot_description/magni/inertial.xacro" />
   <link name="base_link" />
-  <joint name="chassis_joint" type="fixed">
+  <joint name="base_link_to_front_chasis_joint" type="fixed">
     <child link="front_chassis_link"/>
     <parent link="base_link"/>
@@ -123,4 +123,16 @@
       <state_interface name="effort" />
     </joint>
+    <joint name="chassis_joint">
+      <state_interface name="position" />
+      <state_interface name="velocity" />
+    </joint>
+    <joint name="back_right_wheel_joint">
+      <state_interface name="position" />
+      <state_interface name="velocity" />
+    </joint>
+    <joint name="back_left_wheel_joint">
+      <state_interface name="position" />
+      <state_interface name="velocity" />
+    </joint>
   </ros2_control>
   <gazebo>
@@ -144,4 +156,11 @@
       <frame_id>front_chassis_link</frame_id>
     </sensor>
+    <sensor name="imu" type="imu">
+      <always_on>1</always_on>
+      <update_rate>100</update_rate>
+      <visualize>true</visualize>
+      <topic>imu</topic>
+      <enable_metrics>true</enable_metrics>
+    </sensor>
   </gazebo>
 </robot>
